Commit message: time has come.

File: src/haircut/Assembly_copy/Assembly_copy.urdf (robot description, URDF)
Before this commit: robot Assembly_copy, 8 links, 7 joints
Joints:
- joint rev1: limit lower=-1.5 upper=1.5 effort=100 velocity=10 -> lower=-2.5 upper=2.5 effort=100 velocity=10
- joint rev2: limit lower=-1.5 upper=1.5 effort=100 velocity=10 -> lower=-2.5 upper=2.5 effort=100 velocity=10
- joint rev3: limit lower=-1.5 upper=1.5 effort=100 velocity=10 -> lower=-2.5 upper=2.5 effort=100 velocity=10
- joint rev4: limit lower=-1.5 upper=1.5 effort=100 velocity=10 -> lower=-2.5 upper=2.5 effort=100 velocity=10
- joint rev5: limit lower=-1.5 upper=1.5 effort=100 velocity=10 -> lower=-2.5 upper=2.5 effort=100 velocity=10
- joint rev6: limit lower=-1.5 upper=1.5 effort=100 velocity=10 -> lower=-2.5 upper=2.5 effort=100 velocity=10

File: src/haircut/Assembly_copy/hw_Assembly_copy.urdf (robot description, URDF)
Before this commit: robot Assembly_copy, 8 links, 7 joints
Joints:
- joint rev1: limit lower=-1.5 upper=1.5 effort=100 velocity=10 -> lower=-2.5 upper=2.5 effort=100 velocity=10
- joint rev2: limit lower=-1.5 upper=1.5 effort=100 velocity=10 -> lower=-2.5 upper=2.5 effort=100 velocity=10
- joint rev3: limit lower=-1.5 upper=1.5 effort=100 velocity=10 -> lower=-2.5 upper=2.5 effort=100 velocity=10
- joint rev4: limit lower=-1.5 upper=1.5 effort=100 velocity=10 -> lower=-2.5 upper=2.5 effort=100 velocity=10
- joint rev5: limit lower=-1.5 upper=1.5 effort=100 velocity=10 -> lower=-2.5 upper=2.5 effort=100 velocity=10
- joint rev6: limit lower=-1.5 upper=1.5 effort=100 velocity=10 -> lower=-2.5 upper=2.5 effort=100 velocity=10

File: src/haircut/Assembly_copy/hwsim_Assembly_copy.urdf (robot description, URDF)
Before this commit: robot Assembly_copy, 8 links, 7 joints
Joints:
- joint rev1: limit lower=-1.5 upper=1.5 effort=100 velocity=10 -> lower=-2.5 upper=2.5 effort=100 velocity=10
- joint rev2: limit lower=-1.5 upper=1.5 effort=100 velocity=10 -> lower=-2.5 upper=2.5 effort=100 velocity=10
- joint rev3: limit lower=-1.5 upper=1.5 effort=100 velocity=10 -> lower=-2.5 upper=2.5 effort=100 velocity=10
- joint rev4: limit lower=-1.5 upper=1.5 effort=100 velocity=10 -> lower=-2.5 upper=2.5 effort=100 velocity=10
- joint rev5: limit lower=-1.5 upper=1.5 effort=100 velocity=10 -> lower=-2.5 upper=2.5 effort=100 velocity=10
- joint rev6: limit lower=-1.5 upper=1.5 effort=100 velocity=10 -> lower=-2.5 upper=2.5 effort=100 velocity=10
